File: V1.1/ebike_LED.kicad_pcb (KiCad board)
At the start: 2 copper layers, 45.7 x 43.2 mm, 5 parts, among them SW1 SW_Push

Commit message: gerber generation
Parts:
- added R2: 10k, Resistor_SMD:R_0805_2012Metric, F.Cu at (72.4, 47.0)
- added SW2: SW_Push, Button_Switch_THT:SW_PUSH-12mm, F.Cu at (101.8, 52.1)
- R1: renamed from R6; moved to F.Cu
- SW1: footprint Button_Switch_THT:SW_PUSH_6mm_H8mm -> Button_Switch_THT:SW_PUSH-12mm
- moved SW1 53.1 mm to (101.8, 30.4)
- moved R1 17.0 mm to (68.6, 47.0), turned to 90 degrees
Connections:
- A1 pad 25: unconnected-(A1-Pad25) -> PB2_IN
- LED1 pad 1: +3.3v -> Vcc
- LED1 pad 2: Vcc -> +3.3v
Routing:
- net Vcc: track 0.00 -> 87.9 mm, vias 0 -> 1
- net PB1_IN: track 0.00 -> 72.9 mm
- net PB2_IN: track 0.00 -> 57.8 mm, vias 0 -> 1
- net SDA: track 0.00 -> 23.3 mm
- net SCL: track 0.00 -> 22.4 mm
- net TX: track 0.23 -> 5.10 mm
- net RX: track 0.18 -> 5.04 mm
- added copper zone on F.Cu, net +3.3v
- removed copper zone on F.Cu, net Vcc
Other:
- board size 45.7 x 43.2 mm -> 68.6 x 43.2 mm
- board text added: "+3.3"
- board text added: "GND"
- board text added: "RX"
- board text added: "SCL"
- board text added: "SDA"
- board text added: "TX"
- board text added: "Vcc"
