File: speed_joystick/speed_joystick.kicad_pcb (KiCad board)
At the start: 2 copper layers, 89.2 x 61.1 mm, 5 parts, among them U1 Teensy3.2

Commit message: pcb work
Parts:
- added C1: 104, Capacitor_SMD:C_0603_1608Metric, F.Cu at (35.2, 0.76)
- added C10: 104, Capacitor_SMD:C_0603_1608Metric, F.Cu at (39.2, 8.29)
- added C11: 104, Capacitor_SMD:C_0603_1608Metric, F.Cu at (39.2, 10.8)
- added C12: 104, Capacitor_SMD:C_0603_1608Metric, F.Cu at (39.2, 13.3)
- added C13: 104, Capacitor_SMD:C_0603_1608Metric, F.Cu at (43.2, 0.76)
- added C14: 104, Capacitor_SMD:C_0603_1608Metric, F.Cu at (43.2, 3.27)
- added C15: 104, Capacitor_SMD:C_0603_1608Metric, F.Cu at (43.2, 5.78)
- added C16: 104, Capacitor_SMD:C_0603_1608Metric, F.Cu at (43.2, 8.29)
- added C17: 104, Capacitor_SMD:C_0603_1608Metric, F.Cu at (43.2, 10.8)
- added C18: 104, Capacitor_SMD:C_0603_1608Metric, F.Cu at (43.2, 13.3)
- added C19: 104, Capacitor_SMD:C_0603_1608Metric, F.Cu at (47.2, 0.76)
- added C2: 104, Capacitor_SMD:C_0603_1608Metric, F.Cu at (35.2, 3.27)
- added C20: 104, Capacitor_SMD:C_0603_1608Metric, F.Cu at (47.2, 3.27)
- added C21: 104, Capacitor_SMD:C_0603_1608Metric, F.Cu at (47.2, 5.78)
- added C22: 104, Capacitor_SMD:C_0603_1608Metric, F.Cu at (47.2, 8.29)
- added C23: 104, Capacitor_SMD:C_0603_1608Metric, F.Cu at (47.2, 10.8)
- added C24: 104, Capacitor_SMD:C_0603_1608Metric, F.Cu at (47.2, 13.3)
- added C3: 104, Capacitor_SMD:C_0603_1608Metric, F.Cu at (35.2, 5.78)
- added C4: 104, Capacitor_SMD:C_0603_1608Metric, F.Cu at (35.2, 8.29)
- added C5: 104, Capacitor_SMD:C_0603_1608Metric, F.Cu at (35.2, 10.8)
- added C6: 104, Capacitor_SMD:C_0603_1608Metric, F.Cu at (35.2, 13.3)
- added C7: 104, Capacitor_SMD:C_0603_1608Metric, F.Cu at (39.2, 0.76)
- added C8: 104, Capacitor_SMD:C_0603_1608Metric, F.Cu at (39.2, 3.27)
- added C9: 104, Capacitor_SMD:C_0603_1608Metric, F.Cu at (39.2, 5.78)
- added D1: SK6812, LED_SMD:LED_SK6812_PLCC4_5.0x5.0mm_P3.2mm, F.Cu at (3.71, 2.81)
- added D10: SK6812, LED_SMD:LED_SK6812_PLCC4_5.0x5.0mm_P3.2mm, F.Cu at (12.1, 16.1)
- added D11: SK6812, LED_SMD:LED_SK6812_PLCC4_5.0x5.0mm_P3.2mm, F.Cu at (12.1, 22.7)
- added D12: SK6812, LED_SMD:LED_SK6812_PLCC4_5.0x5.0mm_P3.2mm, F.Cu at (12.1, 29.3)
- added D13: SK6812, LED_SMD:LED_SK6812_PLCC4_5.0x5.0mm_P3.2mm, F.Cu at (12.1, 35.9)
- added D14: SK6812, LED_SMD:LED_SK6812_PLCC4_5.0x5.0mm_P3.2mm, F.Cu at (12.1, 42.5)
- added D15: SK6812, LED_SMD:LED_SK6812_PLCC4_5.0x5.0mm_P3.2mm, F.Cu at (20.6, 2.81)
- added D16: SK6812, LED_SMD:LED_SK6812_PLCC4_5.0x5.0mm_P3.2mm, F.Cu at (20.6, 9.43)
- added D17: SK6812, LED_SMD:LED_SK6812_PLCC4_5.0x5.0mm_P3.2mm, F.Cu at (20.6, 16.1)
- added D18: SK6812, LED_SMD:LED_SK6812_PLCC4_5.0x5.0mm_P3.2mm, F.Cu at (20.6, 22.7)
- added D19: SK6812, LED_SMD:LED_SK6812_PLCC4_5.0x5.0mm_P3.2mm, F.Cu at (20.6, 29.3)
- added D2: SK6812, LED_SMD:LED_SK6812_PLCC4_5.0x5.0mm_P3.2mm, F.Cu at (3.71, 9.43)
- added D20: SK6812, LED_SMD:LED_SK6812_PLCC4_5.0x5.0mm_P3.2mm, F.Cu at (20.6, 35.9)
- added D21: SK6812, LED_SMD:LED_SK6812_PLCC4_5.0x5.0mm_P3.2mm, F.Cu at (20.6, 42.5)
- added D22: SK6812, LED_SMD:LED_SK6812_PLCC4_5.0x5.0mm_P3.2mm, F.Cu at (29.0, 2.81)
- added D23: SK6812, LED_SMD:LED_SK6812_PLCC4_5.0x5.0mm_P3.2mm, F.Cu at (29.0, 9.43)
- added D24: SK6812, LED_SMD:LED_SK6812_PLCC4_5.0x5.0mm_P3.2mm, F.Cu at (29.0, 16.1)
- added D3: SK6812, LED_SMD:LED_SK6812_PLCC4_5.0x5.0mm_P3.2mm, F.Cu at (3.71, 16.1)
- added D4: SK6812, LED_SMD:LED_SK6812_PLCC4_5.0x5.0mm_P3.2mm, F.Cu at (3.71, 22.7)
- added D5: SK6812, LED_SMD:LED_SK6812_PLCC4_5.0x5.0mm_P3.2mm, F.Cu at (3.71, 29.3)
- added D6: SK6812, LED_SMD:LED_SK6812_PLCC4_5.0x5.0mm_P3.2mm, F.Cu at (3.71, 35.9)
- added D7: SK6812, LED_SMD:LED_SK6812_PLCC4_5.0x5.0mm_P3.2mm, F.Cu at (3.71, 42.5)
- added D8: SK6812, LED_SMD:LED_SK6812_PLCC4_5.0x5.0mm_P3.2mm, F.Cu at (12.1, 2.81)
- added D9: SK6812, LED_SMD:LED_SK6812_PLCC4_5.0x5.0mm_P3.2mm, F.Cu at (12.1, 9.43)
- added R1: 10k, Resistor_SMD:R_0805_2012Metric, F.Cu at (53.4, 0.97)
- added R1: 10k, Resistor_SMD:R_0805_2012Metric, F.Cu at (100.2, 79.6)
- added R2: 10k, Resistor_SMD:R_0805_2012Metric, F.Cu at (53.4, 3.92)
- added R2: 10k, Resistor_SMD:R_0805_2012Metric, F.Cu at (100.2, 82.6)
- added R3: 10k, Resistor_SMD:R_0805_2012Metric, F.Cu at (100.2, 85.5)
- added R3: 120, Resistor_SMD:R_0805_2012Metric, F.Cu at (53.4, 6.88)
- added R4: 10k, Resistor_SMD:R_0805_2012Metric, F.Cu at (53.4, 9.82)
- added R4: 10k, Resistor_SMD:R_0805_2012Metric, F.Cu at (100.2, 88.5)
- added R5: 10k, Resistor_SMD:R_0805_2012Metric, F.Cu at (100.2, 91.4)
- added R5: 10k, Resistor_SMD:R_0805_2012Metric, F.Cu at (53.4, 12.8)
- added R6: 10k, Resistor_SMD:R_0805_2012Metric, F.Cu at (53.4, 15.7)
- added R7: 10k, Resistor_SMD:R_0805_2012Metric, F.Cu at (53.4, 18.7)
- added SW1: JS5208, JS5208:SW_JS5208, F.Cu at (106.3, 105.2)
- added U2: SN65HVD230, Package_SO:SOIC-8_3.9x4.9mm_P1.27mm, F.Cu at (59.9, 2.73)
Connections:
- net NRST renamed RST
- net Net-(U1-Pad11) renamed RS/DC
- net Net-(U1-Pad12) renamed CS
- net Net-(U1-Pad13) renamed MOSI
- net Net-(U1-Pad20) renamed SCLK
- U1 pad 14: Net-(U1-Pad14) -> unconnected-(U1-12_DIN-Pad14)
- U1 pad 22: Net-(U1-Pad22) -> unconnected-(U1-15_A1_CS_Touch-Pad22)
- U1 pad 23: Net-(U1-Pad23) -> unconnected-(U1-16_A2_SCL0_Touch-Pad23)
- U1 pad 24: Net-(U1-Pad24) -> unconnected-(U1-17_A3_SDA0_Touch-Pad24)
- U1 pad 25: SDA -> unconnected-(U1-18_A4_SDA0_Touch-Pad25)
- U1 pad 26: SCL -> unconnected-(U1-19_A5_SCL0_Touch-Pad26)
- U1 pad 27: Net-(U1-Pad27) -> unconnected-(U1-20_A6_CS_PWM-Pad27)
- U1 pad 28: Net-(U1-Pad28) -> unconnected-(U1-21_A7_RX1_CS_PWM-Pad28)
- U1 pad 29: Net-(U1-Pad29) -> unconnected-(U1-22_A8_Touch_PWM-Pad29)
- U1 pad 30: Net-(U1-Pad30) -> unconnected-(U1-23_A9_Touch_PWM-Pad30)
- U1 pad 32: Net-(U1-Pad32) -> unconnected-(U1-AGND-Pad32)
- U1 pad 33: Net-(U1-Pad33) -> unconnected-(U1-Vin-Pad33)
- U1 pad 5: B2 -> CAN_TX
- U1 pad 6: B5 -> CAN_RX
- U1 pad 9: Net-(U1-Pad9) -> unconnected-(U1-7_RX3_DOUT-Pad9)

Commit message: work on speed_joystick pcb
Parts:
- removed the R1 at (53.4, 0.97)
- removed the R1 at (100.2, 79.6)
- removed the R2 at (53.4, 3.92)
- removed the R2 at (100.2, 82.6)
- removed the R3 at (100.2, 85.5)
- removed the R3 at (53.4, 6.88)
- removed the R4 at (53.4, 9.82)
- removed the R4 at (100.2, 88.5)
- removed the R5 at (100.2, 91.4)
- removed the R5 at (53.4, 12.8)
- removed the REF** at (84.0, 67.0)
- removed the REF** at (84.0, 122.0)
- removed the REF** at (166.0, 122.0)
- removed the REF** at (166.0, 67.0)
- added ?: , , F.Cu at (66.0, 48.3)
- added ?: , , F.Cu at (63.5, 92.7)
- added ?: , , F.Cu at (104.1, 78.7)
- added ?: , , F.Cu at (66.0, 78.7)
- added ?: , , F.Cu at (104.1, 48.3)
- added ?: , , F.Cu at (22.9, 92.7)
- added C25: 0.1uF, Capacitor_SMD:C_0603_1608Metric, F.Cu at (114.3, 71.4)
- added C26: 0.1uF, Capacitor_SMD:C_0603_1608Metric, F.Cu at (114.6, 64.8)
- added C27: 1uF, Capacitor_SMD:C_0603_1608Metric, F.Cu at (127.7, 71.1)
- added C28: 1uF, Capacitor_SMD:C_0603_1608Metric, F.Cu at (128.0, 65.5)
- added C29: 10uF, Capacitor_SMD:C_0603_1608Metric, F.Cu at (113.0, 64.8)
- added C30: 10uF, Capacitor_SMD:C_0603_1608Metric, F.Cu at (112.5, 71.4)
- added J1: Conn_01x08, 8_hole:8_hole, F.Cu at (114.3, 60.0)
- added J2: Conn_01x04, 4pin:my_4_tab_edge, F.Cu at (31.6, 100.5)
- added J3: Conn_01x09, Connector_PinSocket_2.54mm:PinSocket_1x09_P2.54mm_Vertical, F.Cu at (101.6, 73.7)
- added J4: Conn_01x09, Connector_PinSocket_2.54mm:PinSocket_1x09_P2.54mm_Vertical, F.Cu at (63.5, 73.7)
- added R1: 10k, Resistor_SMD:R_0805_2012Metric, F.Cu at (24.6, 61.7)
- added R2: 10k, Resistor_SMD:R_0805_2012Metric, F.Cu at (24.6, 59.2)
- added R3: 120, Resistor_SMD:R_0805_2012Metric, F.Cu at (32.2, 92.8)
- added R4: 10k, Resistor_SMD:R_0805_2012Metric, F.Cu at (24.6, 56.7)
- added R5: 10k, Resistor_SMD:R_0805_2012Metric, F.Cu at (24.6, 51.6)
- added R8: R, Resistor_SMD:R_0805_2012Metric, F.Cu at (124.5, 74.9)
- added REF**: MountingHole_3.2mm_M3, MountingHole:MountingHole_3.2mm_M3, F.Cu at (114.3, 50.3)
- added REF**: MountingHole_3.2mm_M3, MountingHole:MountingHole_3.2mm_M3, F.Cu at (114.3, 76.7)
- added U3: 100k, Package_SO:TSSOP-20_4.4x6.5mm_P0.65mm, F.Cu at (119.7, 68.5)
- added U4: XC6206PxxxMR, Package_TO_SOT_SMD:SOT-23, F.Cu at (128.3, 68.3)
- D1, D10, D11, D12, D13, D14, D15, D16, D17, D18, D19, D2, D20, D21, D22, D23, D24, D3, D4, D5, D6, D7, D8, D9: footprint LED_SMD:LED_SK6812_PLCC4_5.0x5.0mm_P3.2mm -> LED_SMD:my_SK6812
- U1: moved to B.Cu
- moved D3 138.7 mm to (125.4, 82.7), turned to -150 degrees
- moved D2 138.7 mm to (120.0, 84.9), turned to -165 degrees
- moved D4 138.3 mm to (130.0, 79.2), turned to -135 degrees
- moved D1 138.2 mm to (114.3, 85.7), turned to 180 degrees
- moved D5 137.5 mm to (133.5, 74.6), turned to -120 degrees
- moved D6 136.2 mm to (135.7, 69.2), turned to -105 degrees
- moved D8 135.3 mm to (135.7, 57.8), turned to -75 degrees
- moved D7 134.4 mm to (136.5, 63.5), turned to -90 degrees
- moved D9 128.8 mm to (133.5, 52.4), turned to -60 degrees
- moved D10 122.1 mm to (130.0, 47.8), turned to -45 degrees
- moved C3 121.3 mm to (128.9, 82.8), turned to -54 degrees
- moved C2 120.9 mm to (123.5, 85.9), turned to -69 degrees
- moved C4 120.6 mm to (133.4, 78.3), turned to -39 degrees
- moved C1 119.5 mm to (117.3, 87.5), turned to -84 degrees
- moved C5 118.9 mm to (136.6, 72.9), turned to -24 degrees
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Connections:
- C1 pad 1: +3.3v -> R_+5V
- C1 pad 2: GND -> R_GND
- C10 pad 1: +3.3v -> R_+5V
- C10 pad 2: GND -> R_GND
- C11 pad 1: +3.3v -> R_+5V
- C11 pad 2: GND -> R_GND
- C12 pad 1: +3.3v -> R_+5V
- C12 pad 2: GND -> R_GND
- C13 pad 1: +3.3v -> R_+5V
- C13 pad 2: GND -> R_GND
- C14 pad 1: +3.3v -> R_+5V
- C14 pad 2: GND -> R_GND
- C15 pad 1: +3.3v -> R_+5V
- C15 pad 2: GND -> R_GND
- C16 pad 1: +3.3v -> R_+5V
- C16 pad 2: GND -> R_GND
- C17 pad 1: +3.3v -> R_+5V
- C17 pad 2: GND -> R_GND
- C18 pad 1: +3.3v -> R_+5V
- C18 pad 2: GND -> R_GND
- C19 pad 1: +3.3v -> R_+5V
- C19 pad 2: GND -> R_GND
- C2 pad 1: +3.3v -> R_+5V
- C2 pad 2: GND -> R_GND
- C20 pad 1: +3.3v -> R_+5V
- C20 pad 2: GND -> R_GND
- C21 pad 1: +3.3v -> R_+5V
- C21 pad 2: GND -> R_GND
- C22 pad 1: +3.3v -> R_+5V
- C22 pad 2: GND -> R_GND
- C23 pad 1: +3.3v -> R_+5V
- C23 pad 2: GND -> R_GND
- C24 pad 1: +3.3v -> R_+5V
- C24 pad 2: GND -> R_GND
- C3 pad 1: +3.3v -> R_+5V
- C3 pad 2: GND -> R_GND
- C4 pad 1: +3.3v -> R_+5V
- C4 pad 2: GND -> R_GND
- C5 pad 1: +3.3v -> R_+5V
- C5 pad 2: GND -> R_GND
- C6 pad 1: +3.3v -> R_+5V
- C6 pad 2: GND -> R_GND
- C7 pad 1: +3.3v -> R_+5V
- C7 pad 2: GND -> R_GND
- C8 pad 1: +3.3v -> R_+5V
- C8 pad 2: GND -> R_GND
- C9 pad 1: +3.3v -> R_+5V
- C9 pad 2: GND -> R_GND
- D1 pad 1: GND -> R_GND
- D1 pad 3: Net-(D1-VDD) -> R_+5V
- D1 pad 4: Net-(D1-DOUT) -> unconnected-(D1-DOUT-Pad4)
- D10 pad 1: GND -> R_GND
- D10 pad 3: unconnected-(D10-VDD-Pad3) -> R_+5V
- D11 pad 1: GND -> R_GND
- D11 pad 2: Net-(D10-DOUT) -> Net-(D11-DIN)
- D11 pad 3: +3.3v -> R_+5V
- D11 pad 4: Net-(D11-DOUT) -> Net-(D10-DIN)
- D12 pad 1: GND -> R_GND
- D12 pad 2: Net-(D11-DOUT) -> Net-(D12-DIN)
- D12 pad 3: +3.3v -> R_+5V
- D12 pad 4: Net-(D12-DOUT) -> Net-(D11-DIN)
- D13 pad 1: GND -> R_GND
- D13 pad 2: Net-(D12-DOUT) -> Net-(D13-DIN)
- D13 pad 3: +3.3v -> R_+5V
- D13 pad 4: Net-(D13-DOUT) -> Net-(D12-DIN)
- D14 pad 1: GND -> R_GND
- D14 pad 2: Net-(D13-DOUT) -> Net-(D14-DIN)
- D14 pad 3: +3.3v -> R_+5V
- D14 pad 4: unconnected-(D14-DOUT-Pad4) -> Net-(D13-DIN)
- D15 pad 1: GND -> R_GND
- D15 pad 2: unconnected-(D15-DIN-Pad2) -> Net-(D15-DIN)
- D15 pad 3: +3.3v -> R_+5V
- D15 pad 4: Net-(D15-DOUT) -> Net-(D14-DIN)
- D16 pad 1: GND -> R_GND
- D16 pad 2: Net-(D15-DOUT) -> Net-(D16-DIN)
- D16 pad 3: +3.3v -> R_+5V
- D16 pad 4: Net-(D1-DIN) -> Net-(D15-DIN)
- D17 pad 1: GND -> R_GND
- D17 pad 3: unconnected-(D17-VDD-Pad3) -> R_+5V
- D17 pad 4: Net-(D17-DOUT) -> Net-(D16-DIN)
- D18 pad 1: GND -> R_GND
- D18 pad 2: Net-(D17-DOUT) -> Net-(D18-DIN)
- D18 pad 3: unconnected-(D18-VDD-Pad3) -> R_+5V
- D18 pad 4: Net-(D18-DOUT) -> Net-(D17-DIN)
- D19 pad 1: GND -> R_GND
- D19 pad 2: Net-(D18-DOUT) -> Net-(D19-DIN)
- D19 pad 3: +3.3v -> R_+5V
- D19 pad 4: Net-(D19-DOUT) -> Net-(D18-DIN)
- D2 pad 1: GND -> R_GND
- D2 pad 2: Net-(D1-DOUT) -> Net-(D2-DIN)
- D2 pad 3: Net-(D1-VDD) -> R_+5V
- D2 pad 4: Net-(D2-DOUT) -> Net-(D1-DIN)
- D20 pad 1: GND -> R_GND
- D20 pad 2: Net-(D19-DOUT) -> Net-(D20-DIN)
- D20 pad 3: +3.3v -> R_+5V
- D20 pad 4: Net-(D20-DOUT) -> Net-(D19-DIN)
- D21 pad 1: GND -> R_GND
- D21 pad 2: Net-(D20-DOUT) -> Net-(D21-DIN)
- D21 pad 3: +3.3v -> R_+5V
- D21 pad 4: Net-(D21-DOUT) -> Net-(D20-DIN)
- D22 pad 1: GND -> R_GND
- D22 pad 2: Net-(D21-DOUT) -> Net-(D22-DIN)
- D22 pad 3: +3.3v -> R_+5V
- D22 pad 4: unconnected-(D22-DOUT-Pad4) -> Net-(D21-DIN)
- D23 pad 1: GND -> R_GND
- D23 pad 2: unconnected-(D23-DIN-Pad2) -> Net-(D23-DIN)
- D23 pad 3: +3.3v -> R_+5V
- D23 pad 4: Net-(D23-DOUT) -> Net-(D22-DIN)
- D24 pad 1: GND -> R_GND
- D24 pad 2: Net-(D23-DOUT) -> R_DIN
- D24 pad 3: +3.3v -> R_+5V
- D24 pad 4: unconnected-(D24-DOUT-Pad4) -> Net-(D23-DIN)
- D3 pad 1: GND -> R_GND
- D3 pad 2: Net-(D2-DOUT) -> Net-(D3-DIN)
- D3 pad 3: Net-(D1-VDD) -> R_+5V
- D3 pad 4: Net-(D3-DOUT) -> Net-(D2-DIN)
- D4 pad 1: GND -> R_GND
- D4 pad 2: Net-(D3-DOUT) -> Net-(D4-DIN)
- D4 pad 3: unconnected-(D4-VDD-Pad3) -> R_+5V
- D4 pad 4: Net-(D17-DIN) -> Net-(D3-DIN)
- D5 pad 1: GND -> R_GND
- D5 pad 2: unconnected-(D5-DIN-Pad2) -> Net-(D5-DIN)
- D5 pad 3: Net-(D5-VDD) -> R_+5V
- D5 pad 4: Net-(D5-DOUT) -> Net-(D4-DIN)
- D6 pad 1: GND -> R_GND
- D6 pad 2: Net-(D5-DOUT) -> Net-(D6-DIN)
- D6 pad 3: Net-(D5-VDD) -> R_+5V
- D6 pad 4: Net-(D6-DOUT) -> Net-(D5-DIN)
- D7 pad 1: GND -> R_GND
- D7 pad 2: Net-(D6-DOUT) -> Net-(D7-DIN)
- D7 pad 3: Net-(D5-VDD) -> R_+5V
- D7 pad 4: Net-(D7-DOUT) -> Net-(D6-DIN)
- D8 pad 1: GND -> R_GND
- D8 pad 2: Net-(D7-DOUT) -> Net-(D8-DIN)
- D8 pad 3: unconnected-(D8-VDD-Pad3) -> R_+5V
- D8 pad 4: Net-(D8-DOUT) -> Net-(D7-DIN)
- D9 pad 1: GND -> R_GND
- D9 pad 2: Net-(D8-DOUT) -> Net-(D10-DOUT)
- D9 pad 3: unconnected-(D9-VDD-Pad3) -> R_+5V
- D9 pad 4: Net-(D10-DIN) -> Net-(D8-DIN)
- R6 pad 1: +3.3v -> +3.3V
- U1 pad 10: RST -> RES
- U1 pad 11: RS/DC -> DC
- U1 pad 21: P_IN -> unconnected-(U1-14_A0_SCK-Pad21)
- U1 pad 22: unconnected-(U1-15_A1_CS_Touch-Pad22) -> B5
- U1 pad 23: unconnected-(U1-16_A2_SCL0_Touch-Pad23) -> B4
- U1 pad 24: unconnected-(U1-17_A3_SDA0_Touch-Pad24) -> DIN_SIG
- U1 pad 25: unconnected-(U1-18_A4_SDA0_Touch-Pad25) -> B3
- U1 pad 26: unconnected-(U1-19_A5_SCL0_Touch-Pad26) -> B1
- U1 pad 27: unconnected-(U1-20_A6_CS_PWM-Pad27) -> BL
- U1 pad 28: unconnected-(U1-21_A7_RX1_CS_PWM-Pad28) -> B2
- U1 pad 31: +3.3v -> +3.3V
- U1 pad 33: unconnected-(U1-Vin-Pad33) -> +5V
- U1 pad 4: B1 -> unconnected-(U1-2-Pad4)
- U1 pad 7: B4 -> unconnected-(U1-5_TX1_PWM-Pad7)
- U1 pad 8: B3 -> unconnected-(U1-6_PWM-Pad8)
- U2 pad 3: +3.3v -> +3.3V
Routing:
- net +5V: track 0.00 -> 114.8 mm
- net R_+5V: track 0.00 -> 106.6 mm
- net R_GND: track 0.00 -> 69.1 mm, vias 0 -> 53
- net CAN_RX: track 0.00 -> 54.8 mm, vias 0 -> 1
- net CAN_TX: track 0.00 -> 53.5 mm
- net B3: track 0.00 -> 47.5 mm, vias 0 -> 2
- net B4: track 0.00 -> 44.0 mm, vias 0 -> 2
- net B5: track 0.00 -> 41.6 mm, vias 0 -> 2
- net B1: track 0.00 -> 38.4 mm, vias 0 -> 2
- net R_DIN: track 0.00 -> 37.1 mm
- net R_BL: track 0.00 -> 29.9 mm
- net R_RES: track 0.00 -> 27.1 mm
- net B2: track 0.00 -> 25.4 mm
- net R_DC: track 0.00 -> 24.2 mm
- net R_+3.3V: track 0.00 -> 23.7 mm
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- added copper zone on F.Cu, net +3.3V
- added copper zone on F.Cu, net R_+5V
- added copper zone on B.Cu, net R_GND
- removed copper zone on F.Cu, net +3.3v
Other:
- board size 89.2 x 61.1 mm -> 120.2 x 71.1 mm
- board text added: "SPEED JOYSTICK V1.0"

Commit message: created V1.2
Parts:
- removed the ? at (63.5, 92.7)
- removed the ? at (22.9, 92.7)
- removed the REF** at (114.3, 50.3)
- removed the REF** at (114.3, 76.7)
- added ?: , , F.Cu at (-45.8, 0.00)
- added ?: , , F.Cu at (-96.5, 24.6)
- added ?: , , F.Cu at (-49.5, -2.54)
- added ?: , , F.Cu at (-45.7, 24.6)
- added ?: , , F.Cu at (17.8, 0.00)
- added REF**: PinHeader_1x01_P2.54mm_Vertical, Connector_PinHeader_2.54mm:PinHeader_1x01_P2.54mm_Vertical, F.Cu at (14.0, -2.54)
- C1, C10, C11, C12, C13, C14, C15, C16, C17, C18, C19, C2, C20, C21, C22, C23, C24, C3, C4, C5, C6, C7, C8, C9: value 104 -> 0.1uF
- D1, D10, D11, D12, D13, D14, D15, D16, D17, D18, D19, D2, D20, D21, D22, D23, D24, D3, D4, D5, D6, D7, D8, D9: footprint LED_SMD:my_SK6812 -> LED_SMD:LED-SMD_4P-L4.0-W1.6-L
- R3: value 120 -> 10k
- R7: value 10k -> 120
- R8: value R -> 100k
- U2: value SN65HVD230 -> TJA1050T/CM,118
- U3: value 100k -> TXS0108E
- moved ? 153.6 mm to (-73.8, -15.4)
- moved ? 153.6 mm to (-73.8, 15.1)
- moved J4 153.6 mm to (-76.3, 10.0)
- moved C1 134.7 mm to (-0.51, 22.3), turned to 90 degrees
- moved C24 134.6 mm to (-6.27, 21.4), turned to 75 degrees
- moved C2 134.5 mm to (5.29, 21.7), turned to 105 degrees
- moved C23 134.3 mm to (-11.6, 19.1), turned to 60 degrees
- moved C3 134.0 mm to (10.7, 19.6), turned to 120 degrees
- moved C22 133.7 mm to (-16.2, 15.4), turned to 45 degrees
- moved D17 133.5 mm to (-21.5, -12.5), turned to -120 degrees
- moved D18 133.4 mm to (-24.0, -6.50), turned to -105 degrees
- moved C4 133.4 mm to (15.4, 16.2), turned to 135 degrees
- moved D16 133.3 mm to (-17.6, -17.6), turned to -135 degrees
- moved D19 133.1 mm to (-24.9, -0.06), turned to -90 degrees
- moved D15 133.0 mm to (-12.4, -21.6), turned to -150 degrees
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Connections:
- D1 pad 1: R_GND -> Net-(D1-DIN)
- D1 pad 2: Net-(D1-DIN) -> R_+5V
- D1 pad 3: R_+5V -> unconnected-(D1-DOUT-Pad3)
- D1 pad 4: unconnected-(D1-DOUT-Pad4) -> R_GND
- D10 pad 1: R_GND -> Net-(D10-DIN)
- D10 pad 2: Net-(D10-DIN) -> R_+5V
- D10 pad 3: R_+5V -> Net-(D10-DOUT)
- D10 pad 4: Net-(D10-DOUT) -> R_GND
- D11 pad 1: R_GND -> Net-(D11-DIN)
- D11 pad 2: Net-(D11-DIN) -> R_+5V
- D11 pad 3: R_+5V -> Net-(D10-DIN)
- D11 pad 4: Net-(D10-DIN) -> R_GND
- D12 pad 1: R_GND -> Net-(D12-DIN)
- D12 pad 2: Net-(D12-DIN) -> R_+5V
- D12 pad 3: R_+5V -> Net-(D11-DIN)
- D12 pad 4: Net-(D11-DIN) -> R_GND
- D13 pad 1: R_GND -> Net-(D13-DIN)
- D13 pad 2: Net-(D13-DIN) -> R_+5V
- D13 pad 3: R_+5V -> Net-(D12-DIN)
- D13 pad 4: Net-(D12-DIN) -> R_GND
- D14 pad 1: R_GND -> Net-(D14-DIN)
- D14 pad 2: Net-(D14-DIN) -> R_+5V
- D14 pad 3: R_+5V -> Net-(D13-DIN)
- D14 pad 4: Net-(D13-DIN) -> R_GND
- D15 pad 1: R_GND -> Net-(D15-DIN)
- D15 pad 2: Net-(D15-DIN) -> R_+5V
- D15 pad 3: R_+5V -> Net-(D14-DIN)
- D15 pad 4: Net-(D14-DIN) -> R_GND
- D16 pad 1: R_GND -> Net-(D16-DIN)
- D16 pad 2: Net-(D16-DIN) -> R_+5V
- D16 pad 3: R_+5V -> Net-(D15-DIN)
- D16 pad 4: Net-(D15-DIN) -> R_GND
- D17 pad 1: R_GND -> Net-(D17-DIN)
- D17 pad 2: Net-(D17-DIN) -> R_+5V
- D17 pad 3: R_+5V -> Net-(D16-DIN)
- D17 pad 4: Net-(D16-DIN) -> R_GND
- D18 pad 1: R_GND -> Net-(D18-DIN)
- D18 pad 2: Net-(D18-DIN) -> R_+5V
- D18 pad 3: R_+5V -> Net-(D17-DIN)
- D18 pad 4: Net-(D17-DIN) -> R_GND
- D19 pad 1: R_GND -> Net-(D19-DIN)
- D19 pad 2: Net-(D19-DIN) -> R_+5V
- D19 pad 3: R_+5V -> Net-(D18-DIN)
- D19 pad 4: Net-(D18-DIN) -> R_GND
- D2 pad 1: R_GND -> Net-(D2-DIN)
- D2 pad 2: Net-(D2-DIN) -> R_+5V
- D2 pad 3: R_+5V -> Net-(D1-DIN)
- D2 pad 4: Net-(D1-DIN) -> R_GND
- D20 pad 1: R_GND -> Net-(D20-DIN)
- D20 pad 2: Net-(D20-DIN) -> R_+5V
- D20 pad 3: R_+5V -> Net-(D19-DIN)
- D20 pad 4: Net-(D19-DIN) -> R_GND
- D21 pad 1: R_GND -> Net-(D21-DIN)
- D21 pad 2: Net-(D21-DIN) -> R_+5V
- D21 pad 3: R_+5V -> Net-(D20-DIN)
- D21 pad 4: Net-(D20-DIN) -> R_GND
- D22 pad 1: R_GND -> Net-(D22-DIN)
- D22 pad 2: Net-(D22-DIN) -> R_+5V
- D22 pad 3: R_+5V -> Net-(D21-DIN)
- D22 pad 4: Net-(D21-DIN) -> R_GND
- D23 pad 1: R_GND -> Net-(D23-DIN)
- D23 pad 2: Net-(D23-DIN) -> R_+5V
- D23 pad 3: R_+5V -> Net-(D22-DIN)
- D23 pad 4: Net-(D22-DIN) -> R_GND
- D24 pad 1: R_GND -> DIN_SIG
- D24 pad 2: R_DIN -> R_+5V
- D24 pad 3: R_+5V -> Net-(D23-DIN)
- D24 pad 4: Net-(D23-DIN) -> R_GND
- D3 pad 1: R_GND -> Net-(D3-DIN)
- D3 pad 2: Net-(D3-DIN) -> R_+5V
- D3 pad 3: R_+5V -> Net-(D2-DIN)
- D3 pad 4: Net-(D2-DIN) -> R_GND
- D4 pad 1: R_GND -> Net-(D4-DIN)
- D4 pad 2: Net-(D4-DIN) -> R_+5V
- D4 pad 3: R_+5V -> Net-(D3-DIN)
- D4 pad 4: Net-(D3-DIN) -> R_GND
- D5 pad 1: R_GND -> Net-(D5-DIN)
- D5 pad 2: Net-(D5-DIN) -> R_+5V
- D5 pad 3: R_+5V -> Net-(D4-DIN)
- D5 pad 4: Net-(D4-DIN) -> R_GND
- D6 pad 1: R_GND -> Net-(D6-DIN)
- D6 pad 2: Net-(D6-DIN) -> R_+5V
- D6 pad 3: R_+5V -> Net-(D5-DIN)
- D6 pad 4: Net-(D5-DIN) -> R_GND
- D7 pad 1: R_GND -> Net-(D7-DIN)
- D7 pad 2: Net-(D7-DIN) -> R_+5V
- D7 pad 3: R_+5V -> Net-(D6-DIN)
- D7 pad 4: Net-(D6-DIN) -> R_GND
- D8 pad 1: R_GND -> Net-(D8-DIN)
- D8 pad 2: Net-(D8-DIN) -> R_+5V
- D8 pad 3: R_+5V -> Net-(D7-DIN)
- D8 pad 4: Net-(D7-DIN) -> R_GND
- D9 pad 1: R_GND -> Net-(D10-DOUT)
- D9 pad 2: Net-(D10-DOUT) -> R_+5V
- D9 pad 3: R_+5V -> Net-(D8-DIN)
- D9 pad 4: Net-(D8-DIN) -> R_GND
- J2 pad 1: CAN_LO -> GND
- J2 pad 2: CAN_HI -> CAN_LO
- J2 pad 3: GND -> CAN_HI
- R3 pad 1: CAN_LO -> Net-(U2-Rs)
- R3 pad 2: CAN_HI -> GND
- R7 pad 1: Net-(U2-Rs) -> CAN_LO
- R7 pad 2: GND -> CAN_HI
- U1 pad 24: DIN_SIG -> DIN
- U3 pad 13: unconnected-(U3-B7-Pad13) -> DIN_SIG
- U3 pad 8: unconnected-(U3-A7-Pad8) -> R_DIN
Routing:
- net CAN_RX: track 54.8 -> 11.0 mm, vias 1 -> 0
- net CAN_TX: track 53.5 -> 10.5 mm
- net B2: track 25.4 -> 66.0 mm, vias 0 -> 2
- net CAN_HI: track 12.8 -> 52.6 mm
- net CAN_LO: track 12.3 -> 51.1 mm
- net DIN_SIG: track 0.00 -> 34.7 mm, vias 0 -> 3
- net R_+5V: track 106.6 -> 78.3 mm, vias 0 -> 24
- net MOSI: track 5.75 -> 26.8 mm
- net CS: track 5.75 -> 25.5 mm
- net DC: track 5.75 -> 24.3 mm
- net RES: track 5.75 -> 23.8 mm
- net DIN: track 0.00 -> 17.5 mm
- net B1: track 38.4 -> 54.7 mm, vias 2 -> 0
- net BL: track 22.0 -> 6.43 mm, vias 1 -> 0
- net +5V: track 114.8 -> 100.9 mm, vias 0 -> 1
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Other:
- board size 120.2 x 71.1 mm -> 126.6 x 72.8 mm
- board text added: "+5V"
- board text added: "BL"
- board text added: "CS"
- board text added: "DC"
- board text added: "DIN"
- board text added: "GND"
- board text added: "HI"
- board text added: "LO"
- board text added: "MOSI"
- board text added: "RES"
- board text added: "SCLK"
- board text added: "SPEED JOYSTICK V1.2"
- board text removed: "SPEED JOYSTICK V1.0"

Commit message: created V1.2
Routing:
- net (no net): track 0.00 -> 14.4 mm
Changed lines of the file:
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@@
       (net 68 "+5V") (pinfunction "Vin") (pintype "power_in"))
   )
-  (gr_line (start -98.425 -17.145) (end -95.25 -10.16)
-    (stroke (width 0.2) (type default)) (layer "F.Cu"))
-  (gr_line (start -95.25 -10.16) (end -88.9 -13.335)
-    (stroke (width 0.2) (type default)) (layer "F.Cu"))
   (gr_line (start -55.037543 -24.730311) (end -54.079709 -24.381696)
     (stroke (width 0.2) (type solid)) (layer "Edge.Cuts"))
@@
     (effects (font (size 1 1) (thickness 0.15)) (justify left bottom))
   )
+  (segment (start -98.425 -13.97) (end -98.425 -10.795) (width 0.25) (layer "B.Cu") (net 0))
+  (segment (start -92.71 -12.7) (end -92.71 -15.875) (width 0.25) (layer "B.Cu") (net 0))
+  (segment (start -96.52 -8.89) (end -92.71 -12.7) (width 0.25) (layer "B.Cu") (net 0))
+  (segment (start -98.425 -10.795) (end -96.52 -8.89) (width 0.25) (layer "B.Cu") (net 0))
   (segment (start -95.568 30.29) (end -95.504 30.226) (width 0.5) (layer "F.Cu") (net 1))
   (segment (start -48.38 42.2275) (end -48.38 35.934) (width 0.5) (layer "F.Cu") (net 1))

Commit message: finalized speed_joystick V1.2
Parts:
- added R10: 10k, Resistor_SMD:R_0805_2012Metric, F.Cu at (-50.8, 1.27)
- added R9: 10k, Resistor_SMD:R_0805_2012Metric, F.Cu at (-50.2, 5.08)
- moved R7 36.6 mm to (-41.3, -0.64)
Connections:
- net CS renamed CS1
- U1 pad 2: TX_OUT -> CAN_RX
- U1 pad 22: B5 -> unconnected-(U1-15_A1_CS_Touch-Pad22)
- U1 pad 23: B4 -> B5
- U1 pad 24: DIN -> B4
- U1 pad 27: BL -> unconnected-(U1-20_A6_CS_PWM-Pad27)
- U1 pad 3: RX_OUT -> CAN_TX
- U1 pad 4: unconnected-(U1-2-Pad4) -> DIN
- U1 pad 5: CAN_TX -> unconnected-(U1-3_TX_PWM-Pad5)
- U1 pad 6: CAN_RX -> unconnected-(U1-4_RX_PWM-Pad6)
- U1 pad 7: unconnected-(U1-5_TX1_PWM-Pad7) -> BL
- U1 pad 9: unconnected-(U1-7_RX3_DOUT-Pad9) -> CS2
Routing:
- net (no net): track 14.4 -> 0.00 mm
- net CAN_RX: track 11.0 -> 20.4 mm, vias 0 -> 1
- net BL: track 6.43 -> 0.18 mm
- net DIN: track 17.5 -> 23.7 mm
- net CS2: track 0.00 -> 5.34 mm
- net CAN_TX: track 10.5 -> 15.1 mm
- net B4: track 44.0 -> 47.3 mm
- net B5: track 44.9 -> 47.6 mm
- net CS1: track 25.5 -> 28.1 mm
- net DIN_SIG: track 34.7 -> 32.9 mm, vias 3 -> 2
- net CAN_HI: track 52.6 -> 53.2 mm
- net R_+5V: vias 24 -> 0

Commit message: create jlcpcb order
Other:
- board text added: "U2 CAN CHIP = 270"
- board text added: "U3 TXS0108E ANGLE = 0 U4 Voltage Reg = 180"
