File: speed_joystick/speed_joystick.kicad_sch (KiCad schematic)
At the start: 10 parts, among them J1 Conn_01x07, J2 Conn_01x04, SW1 JS5208, U1 Teensy3.2

Commit message: pcb work
Parts:
- removed RV1: R_POT, Potentiometer_SMD:slide_pot, symbol speed_joystick-rescue:R_POT-Device
- added R6, R7: 10k, Resistor_SMD:R_0805_2012Metric, symbol Device:R
- added U2: SN65HVD230, Package_SO:SOIC-8_3.9x4.9mm_P1.27mm, symbol Interface_CAN_LIN:SN65HVD230
- J2: footprint (none) -> Connector_PinSocket_2.54mm:my_4_tab_edge
- R3: value 10k -> 120; Group# 11 -> (none); P/N 755-ESR10EZPF5102 -> (none)
- SW1: footprint Button_Switch_Keyboard:Joy_switch -> JS5208:SW_JS5208
Connections:
- net +3.3v: now also R6.1, U2.3 (VCC); no longer R3.1
- net B1: now also R6.2; no longer R1.2
- net B2: now also R5.2; no longer R2.2
- net B3: now also R4.2; no longer R3.2
- net B4: now also R2.2; no longer R4.2
- net B5: now also R1.2; no longer R5.2
- net CAN_RX: now also U2.4 (R); no longer J2.2 (Pin_2)
- net CAN_TX: now also U2.1 (D); no longer J2.1 (Pin_1)
- net GND: now also R7.2, U2.2 (GND)
- new net: R7.1, U2.8 (Rs)
- new net CAN_HI: J2.2 (Pin_2), R3.2, U2.7 (CANH)
- new net CAN_LO: J2.1 (Pin_1), R3.1, U2.6 (CANL)
Other:
- added sheet LEDs (untitled.kicad_sch)
- note added: "LED BANK"
- moved on the sheet: J1, J2

Commit message: work on speed_joystick pcb
Parts:
- removed J1: Conn_01x07, symbol Connector_Generic:Conn_01x07
- added J4: Conn_01x09, Connector_PinSocket_2.54mm:PinSocket_1x09_P2.54mm_Vertical, symbol Connector_Generic:Conn_01x09
- J2: footprint Connector_PinSocket_2.54mm:my_4_tab_edge -> 4pin:my_4_tab_edge
Connections:
- net RST is gone; now on net RES: U1.10 (8_TX3_DIN)
- net B1: now also U1.26 (19_A5_SCL0_Touch); no longer U1.4 (2)
- net B2: now also U1.28 (21_A7_RX1_CS_PWM)
- net B3: now also U1.25 (18_A4_SDA0_Touch); no longer U1.8 (6_PWM)
- net B4: now also U1.23 (16_A2_SCL0_Touch); no longer U1.7 (5_TX1_PWM)
- net B5: now also U1.22 (15_A1_CS_Touch)
- net CS: now also J4.5 (Pin_5)
- net GND: now also J4.2 (Pin_2)
- net MOSI: now also J4.3 (Pin_3)
- net RES: now also J4.7 (Pin_7)
- net SCLK: now also J4.4 (Pin_4)
- net DIN_SIG: now reaches U1.24 (17_A3_SDA0_Touch)
- net BL: now reaches U1.27 (20_A6_CS_PWM)
- net BL: now also J4.8 (Pin_8)
- net +5V: now reaches U1.33 (Vin)
- net +5V: now also J2.4 (Pin_4), J4.1 (Pin_1)
- net +3.3v renamed +3.3V
- net +3.3V: no longer J2.4 (Pin_4)
- net P_IN: no longer names the net of U1.21 (14_A0_SCK)
- net RS/DC renamed DC
- net DC: now also J4.6 (Pin_6)
- new net DIN: J4.9 (Pin_9)
Other:
- sheet LEDs ports: added +5V, BL, CS, DC, DIN, GND, MOSI, RES, SCLK; removed none
- note removed: "SCL"
- note removed: "SDA"
- moved on the sheet: J2, SW1, U1, U2

Commit message: more round oled work
Parts:
- renumbered R7 to R3, R3 to R7
Changed lines of the file:
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@@
   (symbol (lib_id "Device:R") (at 106.68 86.36 0) (unit 1)
     (in_bom yes) (on_board yes) (dnp no) (fields_autoplaced)
-    (property "Reference" "R7" (at 104.14 86.995 0)
+    (property "Reference" "R3" (at 104.14 86.995 0)
       (effects (font (size 1.27 1.27)) (justify right) hide)
     )
@@
       (project "speed_joystick"
         (path "/4a59a5af-ed4b-4cb8-b8a2-3b43f8ee3aeb"
-          (reference "R7") (unit 1)
+          (reference "R3") (unit 1)
         )
       )
@@
   (symbol (lib_id "Device:R") (at 139.7 80.01 180) (unit 1)
     (in_bom yes) (on_board yes) (dnp no) (fields_autoplaced)
-    (property "Reference" "R3" (at 142.24 79.375 0)
+    (property "Reference" "R7" (at 142.24 79.375 0)
       (effects (font (size 1.27 1.27)) (justify right) hide)
     )
@@
       (project "speed_joystick"
         (path "/4a59a5af-ed4b-4cb8-b8a2-3b43f8ee3aeb"
-          (reference "R3") (unit 1)
+          (reference "R7") (unit 1)
         )
       )

Commit message: created V1.2
Parts:
- R1, R2, R3, R4, R5, R6: LCSC (none) -> C25804
- R7: LCSC (none) -> C17437
- SW1: LCSC (none) -> C3029619
- U2: value SN65HVD230 -> TJA1050T/CM,118; LCSC (none) -> C6952
Connections:
- net DIN_SIG is gone; now on net DIN: U1.24 (17_A3_SDA0_Touch)
- net CAN_HI: now also J2.3 (Pin_3); no longer J2.2 (Pin_2)
- net CAN_LO: now also J2.2 (Pin_2); no longer J2.1 (Pin_1)
- net GND: now also J2.1 (Pin_1); no longer J2.3 (Pin_3)
Other:
- moved on the sheet: J2
Changed lines of the file:
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@@
     )
   )
-  (global_label "+5V" (shape input) (at 161.29 59.055 0) (fields_autoplaced)
-    (effects (font (size 1.27 1.27)) (justify left))
-    (property "Intersheetrefs" "${INTERSHEET_REFS}" (at 167.4121 59.055 0)
+  (global_label "+5V" (shape input) (at 161.29 59.69 0) (fields_autoplaced)
+    (effects (font (size 1.27 1.27)) (justify left))
+    (property "Intersheetrefs" "${INTERSHEET_REFS}" (at 167.4121 59.69 0)
       (effects (font (size 1.27 1.27)) (justify left) hide)
     )
@@
     )
   )
-  (global_label "CAN_LO" (shape input) (at 161.29 66.675 0) (fields_autoplaced)
-    (effects (font (size 1.27 1.27)) (justify left))
-    (property "Intersheetrefs" "${INTERSHEET_REFS}" (at 170.5569 66.675 0)
+  (global_label "CAN_LO" (shape input) (at 161.29 64.77 0) (fields_autoplaced)
+    (effects (font (size 1.27 1.27)) (justify left))
+    (property "Intersheetrefs" "${INTERSHEET_REFS}" (at 170.5569 64.77 0)
       (effects (font (size 1.27 1.27)) (justify left) hide)
     )
@@
     )
   )
-  (global_label "CAN_HI" (shape input) (at 161.29 64.135 0) (fields_autoplaced)
-    (effects (font (size 1.27 1.27)) (justify left))
-    (property "Intersheetrefs" "${INTERSHEET_REFS}" (at 170.1336 64.135 0)
+  (global_label "CAN_HI" (shape input) (at 161.29 62.23 0) (fields_autoplaced)
+    (effects (font (size 1.27 1.27)) (justify left))
+    (property "Intersheetrefs" "${INTERSHEET_REFS}" (at 170.1336 62.23 0)
       (effects (font (size 1.27 1.27)) (justify left) hide)
     )
@@
     )
   )
-  (global_label "GND" (shape input) (at 161.29 61.595 0) (fields_autoplaced)
-    (effects (font (size 1.27 1.27)) (justify left))
-    (property "Intersheetrefs" "${INTERSHEET_REFS}" (at 167.4121 61.595 0)
+  (global_label "GND" (shape input) (at 161.29 67.31 0) (fields_autoplaced)
+    (effects (font (size 1.27 1.27)) (justify left))
+    (property "Intersheetrefs" "${INTERSHEET_REFS}" (at 167.4121 67.31 0)
       (effects (font (size 1.27 1.27)) (justify left) hide)
     )
@@
     )
   )
-  (global_label "DIN_SIG" (shape input) (at 38.481 81.153 180) (fields_autoplaced)
-    (effects (font (size 1.27 1.27)) (justify right))
-    (property "Intersheetrefs" "${INTERSHEET_REFS}" (at 28.9722 81.153 0)
+  (global_label "DIN" (shape input) (at 38.481 81.153 180) (fields_autoplaced)
+    (effects (font (size 1.27 1.27)) (justify right))
+    (property "Intersheetrefs" "${INTERSHEET_REFS}" (at 33.0241 81.153 0)
       (effects (font (size 1.27 1.27)) (justify right) hide)
     )
@@
       (effects (font (size 1.27 1.27)) hide)
     )
+    (property "LCSC" "C3029619" (at 43.18 110.49 0)
+      (effects (font (size 1.27 1.27)) hide)
+    )
     (pin "1")
     (pin "2")
@@
     )
     (property "Group#" "11" (at 52.07 120.65 0)
+      (effects (font (size 1.27 1.27)) hide)
+    )
+    (property "LCSC" "C25804" (at 52.07 120.65 0)
       (effects (font (size 1.27 1.27)) hide)
     )
@@
       (effects (font (size 1.27 1.27)) hide)
     )
+    (property "LCSC" "C25804" (at 106.68 86.36 0)
+      (effects (font (size 1.27 1.27)) hide)
+    )
     (pin "1")
     (pin "2")
@@
       (effects (font (size 1.27 1.27)) hide)
     )
+    (property "LCSC" "C17437" (at 139.7 80.01 0)
+      (effects (font (size 1.27 1.27)) hide)
+    )
     (pin "1")
     (pin "2")
@@
       (effects (font (size 1.27 1.27)) hide)
     )
+    (property "LCSC" "C25804" (at 52.07 125.73 0)
+      (effects (font (size 1.27 1.27)) hide)
+    )
     (pin "1")
     (pin "2")
@@
       (effects (font (size 1.27 1.27)) hide)
     )
+    (property "LCSC" "C25804" (at 52.07 128.27 0)
+      (effects (font (size 1.27 1.27)) hide)
+    )
     (pin "1")
     (pin "2")
@@
       (effects (font (size 1.27 1.27)) (justify left))
     )
-    (property "Value" "SN65HVD230" (at 123.8759 69.85 0)
+    (property "Value" "TJA1050T/CM,118" (at 123.8759 69.85 0)
       (effects (font (size 1.27 1.27)) (justify left))
     )
@@
       (effects (font (size 1.27 1.27)) hide)
     )
-    (property "Datasheet" "http://www.ti.com/lit/ds/symlink/sn65hvd230.pdf" (at 119.38 66.04 0)
+    (property "Datasheet" "https://jlcpcb.com/partdetail/NxpSemicon-TJA1050T_CM118/C6952#:~:text=Datasheet-,Download,-Source" (at 119.38 66.04 0)
+      (effects (font (size 1.27 1.27)) hide)
+    )
+    (property "LCSC" "C6952" (at 121.92 76.2 0)
       (effects (font (size 1.27 1.27)) hide)
     )
@@
     )
   )
-  (symbol (lib_id "Connector_Generic:Conn_01x04") (at 156.21 64.135 180) (unit 1)
+  (symbol (lib_id "Connector_Generic:Conn_01x04") (at 156.21 64.77 180) (unit 1)
     (in_bom yes) (on_board yes) (dnp no) (fields_autoplaced)
-    (property "Reference" "J2" (at 156.21 56.515 0)
+    (property "Reference" "J2" (at 156.21 57.15 0)
       (effects (font (size 1.27 1.27)))
     )
-    (property "Value" "Conn_01x04" (at 156.21 56.515 0)
-      (effects (font (size 1.27 1.27)) hide)
-    )
-    (property "Footprint" "4pin:my_4_tab_edge" (at 156.21 64.135 0)
-      (effects (font (size 1.27 1.27)) hide)
-    )
-    (property "Datasheet" "~" (at 156.21 64.135 0)
+    (property "Value" "Conn_01x04" (at 156.21 57.15 0)
+      (effects (font (size 1.27 1.27)) hide)
+    )
+    (property "Footprint" "4pin:my_4_tab_edge" (at 156.21 64.77 0)
+      (effects (font (size 1.27 1.27)) hide)
+    )
+    (property "Datasheet" "~" (at 156.21 64.77 0)
       (effects (font (size 1.27 1.27)) hide)
     )
@@
       (effects (font (size 1.27 1.27)) hide)
     )
+    (property "LCSC" "C25804" (at 52.07 130.81 0)
+      (effects (font (size 1.27 1.27)) hide)
+    )
     (pin "1")
     (pin "2")
@@
       (effects (font (size 1.27 1.27)) hide)
     )
+    (property "LCSC" "C25804" (at 52.07 123.19 0)
+      (effects (font (size 1.27 1.27)) hide)
+    )

Commit message: finalized speed_joystick V1.2
Parts:
- added R10, R9: 10k, Resistor_SMD:R_0805_2012Metric, symbol Device:R
Connections:
- net RX_OUT is gone; now on net CAN_TX: U1.3 (1_TX1_Touch)
- net TX_OUT is gone; now on net CAN_RX: U1.2 (0_RX1_Touch)
- net +3.3V: now also R10.1, R9.1
- net B4: now also U1.24 (17_A3_SDA0_Touch); no longer U1.23 (16_A2_SCL0_Touch)
- net B5: now also U1.23 (16_A2_SCL0_Touch); no longer U1.22 (15_A1_CS_Touch)
- net BL: now also U1.7 (5_TX1_PWM); no longer U1.27 (20_A6_CS_PWM)
- net CAN_RX: no longer U1.6 (4_RX_PWM)
- net CAN_TX: no longer U1.5 (3_TX_PWM)
- net DIN: now also U1.4 (2); no longer U1.24 (17_A3_SDA0_Touch)
- net CS2: now reaches U1.9 (7_RX3_DOUT)
- net CS2: now also R10.2
- net CS renamed CS1
- net CS1: now also R9.2

Commit message: create jlcpcb order
Parts:
- J2, J4, U1: now left out of the parts list
Changed lines of the file:
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@@
   )
   (symbol (lib_id "teensy:Teensy3.2") (at 63.881 57.023 0) (unit 1)
-    (in_bom yes) (on_board yes) (dnp no)
+    (in_bom no) (on_board yes) (dnp no)
     (property "Reference" "U1" (at 63.881 22.5806 0)
       (effects (font (size 1.524 1.524)))
@@
   )
   (symbol (lib_id "Connector_Generic:Conn_01x09") (at 99.06 32.385 0) (mirror y) (unit 1)
-    (in_bom yes) (on_board yes) (dnp no) (fields_autoplaced)
+    (in_bom no) (on_board yes) (dnp no) (fields_autoplaced)
     (property "Reference" "J4" (at 99.06 19.685 0)
       (effects (font (size 1.27 1.27)))
@@
   )
   (symbol (lib_id "Connector_Generic:Conn_01x04") (at 156.21 64.77 180) (unit 1)
-    (in_bom yes) (on_board yes) (dnp no) (fields_autoplaced)
+    (in_bom no) (on_board yes) (dnp no) (fields_autoplaced)
     (property "Reference" "J2" (at 156.21 57.15 0)
       (effects (font (size 1.27 1.27)))
