File: speed_joystick/untitled.kicad_sch (KiCad schematic)
At the start: 48 parts

Commit message: work on speed_joystick pcb
Parts:
- added C16, C17: 1uF, Capacitor_SMD:C_0603_1608Metric, symbol Device:C_Small
- added C25, C26: 0.1uF, Capacitor_SMD:C_0603_1608Metric, symbol Device:C
- added C29, C30: 10uF, Capacitor_SMD:C_0603_1608Metric, symbol Device:C
- added J1: Conn_01x08, 8_hole:8_hole, symbol Connector_Generic:Conn_01x08
- added J3: Conn_01x09, Connector_PinSocket_2.54mm:PinSocket_1x09_P2.54mm_Vertical, symbol Connector_Generic:Conn_01x09
- added R8: R, Resistor_SMD:R_0805_2012Metric, symbol Device:R
- added U3: XC6206PxxxMR, Package_TO_SOT_SMD:SOT-23, symbol Regulator_Linear:XC6206PxxxMR
- added U3: 100k, Package_SO:TSSOP-20_4.4x6.5mm_P0.65mm, symbol Logic_LevelTranslator:TXS0108EPW
- D1: renamed from D16; footprint LED_SMD:LED_SK6812_PLCC4_5.0x5.0mm_P3.2mm -> LED_SMD:my_SK6812
- D10: renamed from D7; footprint LED_SMD:LED_SK6812_PLCC4_5.0x5.0mm_P3.2mm -> LED_SMD:my_SK6812
- D11: renamed from D6; footprint LED_SMD:LED_SK6812_PLCC4_5.0x5.0mm_P3.2mm -> LED_SMD:my_SK6812
- D12: renamed from D5; footprint LED_SMD:LED_SK6812_PLCC4_5.0x5.0mm_P3.2mm -> LED_SMD:my_SK6812
- D13: renamed from D24; footprint LED_SMD:LED_SK6812_PLCC4_5.0x5.0mm_P3.2mm -> LED_SMD:my_SK6812
- D14: renamed from D23; footprint LED_SMD:LED_SK6812_PLCC4_5.0x5.0mm_P3.2mm -> LED_SMD:my_SK6812
- D15: renamed from D22; footprint LED_SMD:LED_SK6812_PLCC4_5.0x5.0mm_P3.2mm -> LED_SMD:my_SK6812
- D16: renamed from D21; footprint LED_SMD:LED_SK6812_PLCC4_5.0x5.0mm_P3.2mm -> LED_SMD:my_SK6812
- D17: renamed from D20; footprint LED_SMD:LED_SK6812_PLCC4_5.0x5.0mm_P3.2mm -> LED_SMD:my_SK6812
- D18: renamed from D19; footprint LED_SMD:LED_SK6812_PLCC4_5.0x5.0mm_P3.2mm -> LED_SMD:my_SK6812
- D19: renamed from D18; footprint LED_SMD:LED_SK6812_PLCC4_5.0x5.0mm_P3.2mm -> LED_SMD:my_SK6812
- D2: renamed from D15; footprint LED_SMD:LED_SK6812_PLCC4_5.0x5.0mm_P3.2mm -> LED_SMD:my_SK6812
- D20: renamed from D17; footprint LED_SMD:LED_SK6812_PLCC4_5.0x5.0mm_P3.2mm -> LED_SMD:my_SK6812
- D21: renamed from D4; footprint LED_SMD:LED_SK6812_PLCC4_5.0x5.0mm_P3.2mm -> LED_SMD:my_SK6812
- D22: renamed from D3; footprint LED_SMD:LED_SK6812_PLCC4_5.0x5.0mm_P3.2mm -> LED_SMD:my_SK6812
- D23: renamed from D2; footprint LED_SMD:LED_SK6812_PLCC4_5.0x5.0mm_P3.2mm -> LED_SMD:my_SK6812
- D24: renamed from D1; footprint LED_SMD:LED_SK6812_PLCC4_5.0x5.0mm_P3.2mm -> LED_SMD:my_SK6812
- D3: renamed from D14; footprint LED_SMD:LED_SK6812_PLCC4_5.0x5.0mm_P3.2mm -> LED_SMD:my_SK6812
- D4: renamed from D13; footprint LED_SMD:LED_SK6812_PLCC4_5.0x5.0mm_P3.2mm -> LED_SMD:my_SK6812
- D5: renamed from D12; footprint LED_SMD:LED_SK6812_PLCC4_5.0x5.0mm_P3.2mm -> LED_SMD:my_SK6812
- D6: renamed from D11; footprint LED_SMD:LED_SK6812_PLCC4_5.0x5.0mm_P3.2mm -> LED_SMD:my_SK6812
- D7: renamed from D10; footprint LED_SMD:LED_SK6812_PLCC4_5.0x5.0mm_P3.2mm -> LED_SMD:my_SK6812
- D8: renamed from D9; footprint LED_SMD:LED_SK6812_PLCC4_5.0x5.0mm_P3.2mm -> LED_SMD:my_SK6812
- D9: renamed from D8; footprint LED_SMD:LED_SK6812_PLCC4_5.0x5.0mm_P3.2mm -> LED_SMD:my_SK6812
Connections:
- net +3.3v is gone; now on net R_+5V: C1.1, C10.1, C11.1, C12.1, C13.1, C14.1, C15.1, C16.1, C17.1, C18.1, C19.1, C2.1, C20.1, C21.1, C22.1, C23.1, C24.1, C3.1, C4.1, C5.1, C6.1, C7.1, C8.1, C9.1, D1.3 (VDD), D13.3 (VDD), D14.3 (VDD), D15.3 (VDD), D16.3 (VDD), D17.3 (VDD), D18.3 (VDD), D2.3 (VDD), D3.3 (VDD), D4.3 (VDD), D5.3 (VDD), D6.3 (VDD)
- net R_+5V: now reaches D19.3 (VDD)
- net R_+5V: now also D10.3 (VDD), D11.3 (VDD), D12.3 (VDD), D20.3 (VDD), D21.3 (VDD), D22.3 (VDD), D23.3 (VDD), D24.3 (VDD), D7.3 (VDD), D8.3 (VDD), D9.3 (VDD), C17.1, C26.1, C29.1, J1.1 (Pin_1), J3.1 (Pin_1), U3.19 (VCCB), U3.3 (VI)
- net at D1.4 (DOUT): no longer D24.2 (DIN)
- net at D13.4 (DOUT): now also D12.2 (DIN)
- net at D3.4 (DOUT): now also D2.2 (DIN)
- net at D15.4 (DOUT): now also D14.2 (DIN)
- net GND renamed R_GND
- net R_GND: now also C16.2, C17.2, C25.2, C26.2, C29.2, C30.2, J1.2 (Pin_2), J3.2 (Pin_2), U3.1 (GND), U3.11 (GND)
- new net: R8.2, U3.10 (OE)
- new net: J1.8 (Pin_8), U3.14 (B6)
- new net: J1.7 (Pin_7), U3.15 (B5)
- new net: J1.6 (Pin_6), U3.16 (B4)
- new net: J1.5 (Pin_5), U3.17 (B3)
- new net: J1.4 (Pin_4), U3.18 (B2)
- new net: J1.3 (Pin_3), U3.20 (B1)
- new net R_+3.3V: C16.1, C25.1, C30.1, R8.1, U3.2 (VCCA), U3.2 (VO)
- new net R_BL: J3.8 (Pin_8), U3.7 (A6)
- new net R_CS: J3.5 (Pin_5), U3.4 (A3)
- new net R_DC: J3.6 (Pin_6), U3.5 (A4)
- new net R_DIN: D24.2 (DIN), J3.9 (Pin_9)
- new net R_MOSI: J3.3 (Pin_3), U3.1 (A1)
- new net R_RES: J3.7 (Pin_7), U3.6 (A5)
- new net R_SCLK: J3.4 (Pin_4), U3.3 (A2)
Other:
- note added: "+5v"
- note added: "BL"
- note added: "CS"
- note added: "DC"
- note added: "GND"
- note added: "MOSI"
- note added: "RES"
- note added: "SCLK"
- moved on the sheet: C1, C10, C11, C12, C13, C14, C15, C16, C17, C18, C19, C2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

Commit message: more round oled work
Parts:
- C1, C10, C11, C12, C13, C14, C15, C16, C17, C18, C19, C2, C20, C21, C22, C23, C24, C3, C4, C5, C6, C7, C8, C9: value 104 -> 0.1uF
- R8: value R -> 100k
Changed lines of the file:
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@@
       (effects (font (size 1.27 1.27)) (justify left))
     )
-    (property "Value" "104" (at 156.0068 86.36 0)
+    (property "Value" "0.1uF" (at 156.0068 86.36 0)
       (effects (font (size 1.27 1.27)) (justify left))
     )
@@
       (effects (font (size 1.27 1.27)) (justify left))
     )
-    (property "Value" "104" (at 103.9368 86.36 0)
+    (property "Value" "0.1uF" (at 103.9368 86.36 0)
       (effects (font (size 1.27 1.27)) (justify left))
     )
@@
       (effects (font (size 1.27 1.27)) (justify left))
     )
-    (property "Value" "104" (at 96.3168 86.36 0)
+    (property "Value" "0.1uF" (at 96.3168 86.36 0)
       (effects (font (size 1.27 1.27)) (justify left))
     )
@@
       (effects (font (size 1.27 1.27)) (justify left))
     )
-    (property "Value" "104" (at 194.1068 86.36 0)
+    (property "Value" "0.1uF" (at 194.1068 86.36 0)
       (effects (font (size 1.27 1.27)) (justify left))
     )
@@
       (effects (font (size 1.27 1.27)) (justify left))
     )
-    (property "Value" "104" (at 201.7268 86.36 0)
+    (property "Value" "0.1uF" (at 201.7268 86.36 0)
       (effects (font (size 1.27 1.27)) (justify left))
     )
@@
       (effects (font (size 1.27 1.27)) (justify left))
     )
-    (property "Value" "104" (at 140.7668 86.36 0)
+    (property "Value" "0.1uF" (at 140.7668 86.36 0)
       (effects (font (size 1.27 1.27)) (justify left))
     )
@@
       (effects (font (size 1.27 1.27)) (justify left))
     )
-    (property "Value" "104" (at 73.4568 86.36 0)
+    (property "Value" "0.1uF" (at 73.4568 86.36 0)
       (effects (font (size 1.27 1.27)) (justify left))
     )
@@
       (effects (font (size 1.27 1.27)) (justify left))
     )
-    (property "Value" "104" (at 163.6268 86.36 0)
+    (property "Value" "0.1uF" (at 163.6268 86.36 0)
       (effects (font (size 1.27 1.27)) (justify left))
     )
@@
       (effects (font (size 1.27 1.27)) (justify left))
     )
-    (property "Value" "104" (at 88.6968 86.36 0)
+    (property "Value" "0.1uF" (at 88.6968 86.36 0)
       (effects (font (size 1.27 1.27)) (justify left))
     )
@@
       (effects (font (size 1.27 1.27)) (justify left))
     )
-    (property "Value" "104" (at 118.11 86.36 0)
+    (property "Value" "0.1uF" (at 118.11 86.36 0)
       (effects (font (size 1.27 1.27)) (justify left))
     )
@@
       (effects (font (size 1.27 1.27)) (justify left))
     )
-    (property "Value" "104" (at 148.3868 86.36 0)
+    (property "Value" "0.1uF" (at 148.3868 86.36 0)
       (effects (font (size 1.27 1.27)) (justify left))
     )
@@
       (effects (font (size 1.27 1.27)) (justify left))
     )
-    (property "Value" "104" (at 111.5568 86.36 0)
+    (property "Value" "0.1uF" (at 111.5568 86.36 0)
       (effects (font (size 1.27 1.27)) (justify left))
     )
@@
       (effects (font (size 1.27 1.27)) (justify left))
     )
-    (property "Value" "104" (at 171.2468 86.36 0)
+    (property "Value" "0.1uF" (at 171.2468 86.36 0)
       (effects (font (size 1.27 1.27)) (justify left))
     )
@@
       (effects (font (size 1.27 1.27)) (justify left))
     )
-    (property "Value" "104" (at 42.9768 86.36 0)
+    (property "Value" "0.1uF" (at 42.9768 86.36 0)
       (effects (font (size 1.27 1.27)) (justify left))
     )
@@
       (effects (font (size 1.27 1.27)) (justify left))
     )
-    (property "Value" "104" (at 186.4868 86.36 0)
+    (property "Value" "0.1uF" (at 186.4868 86.36 0)
       (effects (font (size 1.27 1.27)) (justify left))
     )
@@
       (effects (font (size 1.27 1.27)) (justify left))
     )
-    (property "Value" "104" (at 35.3568 86.36 0)
+    (property "Value" "0.1uF" (at 35.3568 86.36 0)
       (effects (font (size 1.27 1.27)) (justify left))
     )
@@
       (effects (font (size 1.27 1.27)) (justify left))
     )
-    (property "Value" "104" (at 65.8368 86.36 0)
+    (property "Value" "0.1uF" (at 65.8368 86.36 0)
       (effects (font (size 1.27 1.27)) (justify left))
     )
@@
       (effects (font (size 1.27 1.27)) (justify left))
     )
-    (property "Value" "R" (at 158.75 121.285 0)
+    (property "Value" "100k" (at 158.75 121.285 0)
       (effects (font (size 1.27 1.27)) (justify left))
     )
@@
       (effects (font (size 1.27 1.27)) (justify left))
     )
-    (property "Value" "104" (at 81.0768 86.36 0)
+    (property "Value" "0.1uF" (at 81.0768 86.36 0)
       (effects (font (size 1.27 1.27)) (justify left))
     )
@@
       (effects (font (size 1.27 1.27)) (justify left))
     )
-    (property "Value" "104" (at 50.5968 86.36 0)
+    (property "Value" "0.1uF" (at 50.5968 86.36 0)
       (effects (font (size 1.27 1.27)) (justify left))
     )
@@
       (effects (font (size 1.27 1.27)) (justify left))
     )
-    (property "Value" "104" (at 27.7368 86.36 0)
+    (property "Value" "0.1uF" (at 27.7368 86.36 0)
       (effects (font (size 1.27 1.27)) (justify left))
     )
@@
       (effects (font (size 1.27 1.27)) (justify left))
     )
-    (property "Value" "104" (at 58.2168 86.36 0)
+    (property "Value" "0.1uF" (at 58.2168 86.36 0)
       (effects (font (size 1.27 1.27)) (justify left))
     )
@@
       (effects (font (size 1.27 1.27)) (justify left))
     )
-    (property "Value" "104" (at 178.8668 86.36 0)
+    (property "Value" "0.1uF" (at 178.8668 86.36 0)
       (effects (font (size 1.27 1.27)) (justify left))
     )
@@
       (effects (font (size 1.27 1.27)) (justify left))
     )
-    (property "Value" "104" (at 133.1468 86.36 0)
+    (property "Value" "0.1uF" (at 133.1468 86.36 0)
       (effects (font (size 1.27 1.27)) (justify left))
     )
@@
       (effects (font (size 1.27 1.27)) (justify left))
     )
-    (property "Value" "104" (at 125.5268 86.36 0)
-      (effects (font (size 1.27 1.27)) (justify left))
-    )
+    (property "Value" "0.1uF" (at 125.5268 86.36 0)
+      (effects (font (size 1.27 1.27)) (justify left))
+    )

Commit message: created V1.2
Parts:
- C1, C10, C11, C12, C13, C14, C15, C16, C17, C18, C19, C2, C20, C21, C22, C23, C24, C25, C26, C3, C4, C5, C6, C7, C8, C9: LCSC (none) -> C28233
- C29, C30: LCSC (none) -> C96446
- D1, D10, D11, D12, D13, D14, D15, D16, D17, D18, D19, D2, D20, D21, D22, D23, D24, D3, D4, D5, D6, D7, D8, D9: footprint LED_SMD:my_SK6812 -> LED_SMD:LED-SMD_4P-L4.0-W1.6-L; LCSC (none) -> C2890037
- R8: LCSC (none) -> C25803
- U3: value 100k -> TXS0108E; LCSC (none) -> C17206
Connections:
- net R_+5V: now also D1.2 (VDD), D10.2 (VDD), D11.2 (VDD), D12.2 (VDD), D13.2 (VDD), D14.2 (VDD), D15.2 (VDD), D16.2 (VDD), D17.2 (VDD), D18.2 (VDD), D19.2 (VDD), D2.2 (VDD), D20.2 (VDD), D21.2 (VDD), D22.2 (VDD), D23.2 (VDD), D24.2 (VDD), D3.2 (VDD), D4.2 (VDD), D5.2 (VDD), D6.2 (VDD), D7.2 (VDD), D8.2 (VDD), D9.2 (VDD); no longer D1.3 (VDD), D10.3 (VDD), D11.3 (VDD), D12.3 (VDD), D13.3 (VDD), D14.3 (VDD), D15.3 (VDD), D16.3 (VDD), D17.3 (VDD), D18.3 (VDD), D19.3 (VDD), D2.3 (VDD), D20.3 (VDD), D21.3 (VDD), D22.3 (VDD), D23.3 (VDD), D24.3 (VDD), D3.3 (VDD), D4.3 (VDD), D5.3 (VDD), D6.3 (VDD), D7.3 (VDD), D8.3 (VDD), D9.3 (VDD)
- net R_DIN: now also U3.8 (A7); no longer D24.2 (DIN)
- net R_GND: now also D1.4 (VSS), D10.4 (VSS), D11.4 (VSS), D12.4 (VSS), D13.4 (VSS), D14.4 (VSS), D15.4 (VSS), D16.4 (VSS), D17.4 (VSS), D18.4 (VSS), D19.4 (VSS), D2.4 (VSS), D20.4 (VSS), D21.4 (VSS), D22.4 (VSS), D23.4 (VSS), D24.4 (VSS), D3.4 (VSS), D4.4 (VSS), D5.4 (VSS), D6.4 (VSS), D7.4 (VSS), D8.4 (VSS), D9.4 (VSS); no longer D1.1 (VSS), D10.1 (VSS), D11.1 (VSS), D12.1 (VSS), D13.1 (VSS), D14.1 (VSS), D15.1 (VSS), D16.1 (VSS), D17.1 (VSS), D18.1 (VSS), D19.1 (VSS), D2.1 (VSS), D20.1 (VSS), D21.1 (VSS), D22.1 (VSS), D23.1 (VSS), D24.1 (VSS), D3.1 (VSS), D4.1 (VSS), D5.1 (VSS), D6.1 (VSS), D7.1 (VSS), D8.1 (VSS), D9.1 (VSS)
- net DIN_SIG: now reaches U3.13 (B7)
- net DIN_SIG: now also D24.1 (DIN)
- new net: D17.1 (DIN), D18.3 (DOUT)
- new net: D16.1 (DIN), D17.3 (DOUT)
- new net: D19.1 (DIN), D20.3 (DOUT)
- new net: D18.1 (DIN), D19.3 (DOUT)
- new net: D23.1 (DIN), D24.3 (DOUT)
- new net: D22.1 (DIN), D23.3 (DOUT)
- new net: D13.1 (DIN), D14.3 (DOUT)
- new net: D12.1 (DIN), D13.3 (DOUT)
- new net: D11.1 (DIN), D12.3 (DOUT)
- new net: D10.1 (DIN), D11.3 (DOUT)
- new net: D3.1 (DIN), D4.3 (DOUT)
- new net: D2.1 (DIN), D3.3 (DOUT)
- new net: D15.1 (DIN), D16.3 (DOUT)
- new net: D14.1 (DIN), D15.3 (DOUT)
- new net: D1.1 (DIN), D2.3 (DOUT)
- new net: D5.1 (DIN), D6.3 (DOUT)
- new net: D4.1 (DIN), D5.3 (DOUT)
- new net: D10.3 (DOUT), D9.1 (DIN)
- new net: D7.1 (DIN), D8.3 (DOUT)
- new net: D6.1 (DIN), D7.3 (DOUT)
- new net: D21.1 (DIN), D22.3 (DOUT)
- new net: D20.1 (DIN), D21.3 (DOUT)
- new net: D8.1 (DIN), D9.3 (DOUT)

Commit message: create jlcpcb order
Parts:
- J1, J3: now left out of the parts list
Changed lines of the file:
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@@
   )
   (symbol (lib_id "Connector_Generic:Conn_01x09") (at 135.89 146.05 0) (unit 1)
-    (in_bom yes) (on_board yes) (dnp no) (fields_autoplaced)
+    (in_bom no) (on_board yes) (dnp no) (fields_autoplaced)
     (property "Reference" "J3" (at 135.89 133.35 0)
       (effects (font (size 1.27 1.27)))
@@
   )
   (symbol (lib_id "Connector_Generic:Conn_01x08") (at 191.77 138.43 0) (unit 1)
-    (in_bom yes) (on_board yes) (dnp no)
+    (in_bom no) (on_board yes) (dnp no)
     (property "Reference" "J1" (at 191.77 128.27 0)
       (effects (font (size 1.27 1.27)))
