File: mechanical_speedo/mechanical_speedo.kicad_pcb (KiCad board)
At the start: 2 copper layers, 47.8 x 62.2 mm, 31 parts, among them J1 Conn_01x08, J2 Conn_01x04, J3 Conn_01x03, J4 Conn_01x03, SW1 JS5208, U1 Teensy4.0, U2 TJA1050T/CM,118, U3 L6234PD, U6 LD1117S18TR_SOT223

Commit message: added encoder board to mechanical_speedo
Parts:
- added C8: 100nF, Capacitor_SMD:C_0603_1608Metric, F.Cu at (113.3, 79.8)
- added IC1: TLE5012B, TLE5012:SOIC127P600X175-8N, F.Cu at (113.2, 75.2)
- added J5: Conn_01x03, Connector_PinHeader_2.54mm:PinHeader_1x03_P2.54mm_Vertical, F.Cu at (110.7, 70.2)
- added R11: 2.2k, Resistor_SMD:R_0603_1608Metric, F.Cu at (109.7, 75.1)
Connections:
- U1 pad 5: unconnected-(U1-3_LRCLK2-Pad5) -> MOT_ENB
- U3 pad 13: +3.3V -> MOT_ENB
- U3 pad 3: +3.3V -> MOT_ENB
- U3 pad 8: +3.3V -> MOT_ENB
Routing:
- net MOT_ENB: track 0.00 -> 46.6 mm, vias 0 -> 3
- net GND: track 36.5 -> 49.3 mm
- net TLE_PWM: track 0.00 -> 10.6 mm, vias 0 -> 1
- net +3.3V: track 5.33 -> 8.28 mm
Other:
- board size 47.8 x 62.2 mm -> 85 x 62.2 mm
- board text added: "100nF"
- board text added: "3.3v"
- board text added: "PWM"
- board text added: "opt."
